File: Dual_BPF.kicad_pcb (KiCad board)
At the start: 2 copper layers, 150 x 130 mm, 270 parts, among them J1 Conn_Coaxial, J2 Conn_Coaxial, J3 Conn_02x05_Odd_Even, J4 Conn_Coaxial, J5 Conn_Coaxial, J6 Conn_02x05_Odd_Even, K1 EC2-12NU, K10 EC2-12NU, K11 EC2-12NU, K12 EC2-12NU, K13 EC2-12NU, K14 EC2-12NU, K15 EC2-12NU, K16 EC2-12NU, K17 EC2-12NU, K18 EC2-12NU, K19 EC2-12NU, K2 EC2-12NU, K20 EC2-12NU, K21 EC2-12NU, K22 EC2-12NU, K23 EC2-12NU, K24 EC2-12NU, K25 EC2-12NU, K26 EC2-12NU, K27 EC2-12NU, K28 EC2-12NU, K29 EC2-12NU, K3 EC2-12NU, K30 EC2-12NU, K4 EC2-12NU, K5 EC2-12NU, K6 EC2-12NU, K7 EC2-12NU, K8 EC2-12NU, K9 EC2-12NU, Q1 BSP250 /ZVP2106, Q2 BSP250 /ZVP2106, U1 PGA-103, U2 PGA-103

Commit message: SMD version RTM 1.0, toroid version deleted
Parts:
- removed C1, C10, C11, C12, C13, C14, C2, C3, C39, C4, C40, C41, C42, C43, C44, C45, C46, C47, C48, C49, C5, C50, C51, C52, C53, C54, C6, C7, C8, C9: 10n, Capacitor_SMD:C_0805_2012Metric_Pad1.18x1.45mm_HandSolder
- removed C15, C17, C25: 100p, Capacitor_SMD:C_0805_2012Metric_Pad1.18x1.45mm_HandSolder
- removed C16, C19, C27, C38: 100n, Capacitor_SMD:C_0805_2012Metric_Pad1.18x1.45mm_HandSolder
- removed C18, C21, C34, C37: 470p, Capacitor_SMD:C_0805_2012Metric_Pad1.18x1.45mm_HandSolder
- removed C20, C33: 1n, Capacitor_SMD:C_0805_2012Metric_Pad1.18x1.45mm_HandSolder
- removed C22, C35: 270p, Capacitor_SMD:C_0805_2012Metric_Pad1.18x1.45mm_HandSolder
- removed C23, C24, C32, C36: 220p, Capacitor_SMD:C_0805_2012Metric_Pad1.18x1.45mm_HandSolder
- removed C26: 390p, Capacitor_SMD:C_0805_2012Metric_Pad1.18x1.45mm_HandSolder
- removed C28: 680p, Capacitor_SMD:C_0805_2012Metric_Pad1.18x1.45mm_HandSolder
- removed C29: 180p, Capacitor_SMD:C_0805_2012Metric_Pad1.18x1.45mm_HandSolder
- removed C30: 82p, Capacitor_SMD:C_0805_2012Metric_Pad1.18x1.45mm_HandSolder
- removed C31: 47p, Capacitor_SMD:C_0805_2012Metric_Pad1.18x1.45mm_HandSolder
- removed D1: SS36, Diode_SMD:D_SMB
- removed FB1, FB10, FB11, FB12, FB13, FB14, FB15, FB16, FB17, FB18, FB19, FB2, FB20, FB21, FB22, FB23, FB24, FB25, FB26, FB27, FB28, FB29, FB3, FB30, FB4, FB5, FB6, FB7, FB8, FB9: Ferrite, Inductor_SMD:L_0805_2012Metric
- removed H1, H2, H3, H4: MountingHole_Pad, MountingHole:MountingHole_3.2mm_M3_ISO14580_Pad
- removed J1, J2: Conn_Coaxial, SMA_PINS:SMA_PINS
- removed J3: Conn_02x05_Odd_Even, Connector_IDC:IDC-Header_2x05_P2.54mm_Vertical
- removed K1, K10, K11, K12, K13, K14, K15, K2, K3, K4, K5, K6, K7, K8, K9: EC2-12NU, Relay_THT:Relay_DPDT_Kemet_EC2
- removed L1, L15, L5, L7: 330n, Amidon_T50:T50_V_THT_1812_merge
- removed L10: 1u, Amidon_T50:T50_V_THT_1812_merge
- removed L11, L14, L4: 680n, Amidon_T50:T50_V_THT_1812_merge
- removed L12, L17, L2: 10u, Amidon_T50:T50_V_THT_1812_merge
- removed L13, L3, L9: 1.8u, Amidon_T50:T50_V_THT_1812_merge
- removed L16, L6: 150n, Amidon_T50:T50_V_THT_1812_merge
- removed L8: 2.7u, Amidon_T50:T50_V_THT_1812_merge
- removed Q1: BSP250 /ZVP2106, Package_TO_SOT_SMD:SOT-223-3_TabPin2
- removed R1: 10k, Resistor_SMD:R_0805_2012Metric_Pad1.20x1.40mm_HandSolder
- removed R2, R3, R5, R9: 100R, Resistor_SMD:R_0805_2012Metric_Pad1.20x1.40mm_HandSolder
- removed R4, R6, R7: 62R, Resistor_SMD:R_0805_2012Metric_Pad1.20x1.40mm_HandSolder
- removed R8: 30R, Resistor_SMD:R_0805_2012Metric_Pad1.20x1.40mm_HandSolder
- removed U1: PGA-103, Package_TO_SOT_SMD:SOT-89-3
- added REF**: KiCad-Logo2_5mm_SilkScreen, Symbol:KiCad-Logo2_5mm_SilkScreen, F.Cu at (89.5, 112.2)
- added REF**: OSHW-Logo2_7.3x6mm_SilkScreen, Symbol:OSHW-Logo2_7.3x6mm_SilkScreen, F.Cu at (92.8, 32.0)
- FB48, FB50, FB52, FB54, FB56, FB58, FB60: moved to B.Cu
- moved R14 202.3 mm to (78.6, 78.6), turned to 90 degrees
- moved FB41 134.2 mm to (44.0, 70.5), turned to -90 degrees
- moved FB43 131.7 mm to (43.8, 91.2), turned to -90 degrees
- moved FB31 127.1 mm to (44.0, 78.8), turned to -90 degrees
- moved FB46 108.9 mm to (66.5, 101.0), turned to 90 degrees
- moved FB45 108.2 mm to (66.5, 105.2), turned to 90 degrees
- moved FB48 101.1 mm to (98.0, 39.0), turned to 90 degrees
- moved FB50 99.8 mm to (97.8, 47.0), turned to 90 degrees
- moved FB52 98.1 mm to (98.0, 55.0), turned to 90 degrees
- moved FB54 97.0 mm to (97.8, 63.0), turned to 90 degrees
- moved J4 94.4 mm to (72.5, 114.0)
- moved FB60 91.3 mm to (97.8, 79.0), turned to 90 degrees
- moved FB56 90.1 mm to (98.0, 71.0), turned to 90 degrees
- moved FB59 89.1 mm to (98.0, 82.8), turned to -90 degrees
- moved FB55 88.3 mm to (98.0, 74.5), turned to -90 degrees
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Connections:
- net 1.5HPF renamed 1.5HPF_2
- net 13HPF renamed 13HPF_2
- net 20HPF renamed 20HPF_2
- net 6.5HPF renamed 6.5HPF_2
- net 6mLNA renamed 6mLNA_2
- net 9.5HPF renamed 9.5HPF_2
- net HPF_ByPass renamed HPF_ByPass_2
- net RX2_GND renamed RX2_GND_2
Routing:
- net +12V: track 125.6 -> 292.0 mm, vias 6 -> 7
- net 6mLNA_2: track 24.9 -> 118.4 mm
- net GND: track 119.5 -> 38.1 mm, vias 0 -> 376
- net HPF_ByPass_2: track 22.1 -> 88.3 mm, vias 0 -> 2
- net Net-(K14-Pad4): track 56.8 -> 0.00 mm
- net 20HPF_2: track 38.1 -> 88.0 mm
- net 6.5HPF_2: track 84.9 -> 123.1 mm
- net Net-(C23-Pad1): track 31.2 -> 0.00 mm
- net Net-(C21-Pad1): track 29.9 -> 0.00 mm
- net 1.5HPF_2: track 103.9 -> 131.5 mm, vias 0 -> 1
- net Net-(C20-Pad1): track 26.4 -> 0.00 mm
- net Net-(C22-Pad1): track 25.6 -> 0.00 mm
- net RX2_GND_2: track 51.0 -> 26.3 mm, vias 0 -> 1
- net Net-(K30-Pad4): track 0.00 -> 15.0 mm
- net Net-(D2-A): track 0.00 -> 14.9 mm, vias 0 -> 4
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Other:
- board size 150 x 130 mm -> 65 x 90 mm
- board text added: "Alexiares V2 Band Pass Filter"
- board text added: "Schematic KE9H/K6PH Drawing f6itu"
- board text added: "TO_RX1 PS_BOARD / RX2_Ant"
- board text added: "To Alexandrie V2"
- board text added: "To RX1 RX2 Cerberus"
- board text added: "Ἀλεξιάρης"

Commit message: silk done
Other:
- board text added: "+12V RX2 1.5M 9.5M 20M"
- board text added: "GND Bypass 6m LNA 6.5MHz 13MHz"
- board text added: "Sur les bords du ru voisin, campaient deux Huns; non loin d'eux un Gaulois, Eduen peut-être, trempait audacieusement ses pieds dans l'eau courante et fraîche. Sur l'horizon se dessinaient les silhouettes molles de Romains fatigués, de Sarrasins de Corinthe, de Francs anciens, d'Alains seuls. Quelques Normands buvaient du calva. Les Huns préparaient des stèques tartares, le Gaulois fumait une gita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"
Changed lines of the file:
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@@
     (effects (font (size 1 1) (thickness 0.15)) (justify left bottom mirror))
+  )
+  (gr_text "+12V\nRX2\n1.5M\n9.5M\n20M\n" (at 95.9 101.8 90) (layer "B.SilkS")
+    (effects (font (size 1.5 1.5) (thickness 0.3) bold) (justify right bottom mirror))
   )
   (gr_text " Ἀλεξιάρης " (at 78 37.5) (layer "B.SilkS")
     (effects (font (size 2 2) (thickness 0.4) bold) (justify left bottom mirror))
   )
-  (gr_text "To Alexandrie V2" (at 95.5 111) (layer "B.SilkS")
+  (gr_text "To Alexandrie V2" (at 97.7 96.5 90) (layer "B.SilkS")
     (effects (font (size 1 1) (thickness 0.15)) (justify left bottom mirror))
   )
+  (gr_text "Sur les bords du ru voisin, campaient deux Huns; \nnon loin d'eux un Gaulois, Eduen peut-être, \ntrempait audacieusement ses pieds dans l'eau courante et fraîche. \nSur l'horizon se dessinaient les silhouettes molles \nde Romains fatigués, \nde Sarrasins de Corinthe, \nde Francs anciens, \nd'Alains seuls. \nQuelques Normands buvaient du calva.\n\nLes Huns préparaient des stèques tartares, \nle Gaulois fumait une gitane, \nles Romains dessinaient des grecques, \nles Sarrasins fauchaient de l'avoine, \nles Francs cherchaient des sols et les Alains regardaient cinq Ossètes. \nLes Normands buvaient du calva.\n" (at 83.5 41.4 90) (layer "B.SilkS")
+    (effects (font (size 1 1) (thickness 0.15) italic) (justify left bottom mirror))
+  )
+  (gr_text "GND\nBypass\n6m LNA\n6.5MHz\n13MHz\n\n" (at 98 106.7 90) (layer "B.SilkS")
+    (effects (font (size 1.5 1.5) (thickness 0.3) bold) (justify left bottom mirror))
+  )
   (gr_text "To Alexandrie V2" (at 81.5 99) (layer "F.SilkS")
